File: bme280.kicad_sch (KiCad schematic)
At the start: 1 part

Commit message: make board
Connections:
- net +3V3 renamed VIN
Changed lines of the file:
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@@
     (effects (font (size 1.27 1.27)) (justify right))
   )
-  (symbol (lib_id "power:+3V3") (at 128.27 100.33 0) (unit 1)
-    (in_bom yes) (on_board yes) (dnp no) (fields_autoplaced)
-    (property "Reference" "#PWR013" (at 128.27 104.14 0)
-      (effects (font (size 1.27 1.27)) hide)
-    )
-    (property "Value" "+3V3" (at 128.27 95.25 0)
-      (effects (font (size 1.27 1.27)))
-    )
-    (property "Footprint" "" (at 128.27 100.33 0)
-      (effects (font (size 1.27 1.27)) hide)
-    )
-    (property "Datasheet" "" (at 128.27 100.33 0)
-      (effects (font (size 1.27 1.27)) hide)
-    )
-    (pin "1")
-    (instances
-      (project "balloon"
-        (path "/390c33b5-3f3b-4c86-a202-e8d785058178/5b847e45-25d8-440e-b23a-c967243df159"
-          (reference "#PWR013") (unit 1)
-        )
-      )
-    )
+  (hierarchical_label "VIN" (shape input) (at 128.27 100.33 90) (fields_autoplaced)
+    (effects (font (size 1.27 1.27)) (justify left))
   )
   (symbol (lib_id "balloon_lib:BME280") (at 124.46 110.49 0) (unit 1)
