File: bno055.kicad_sch (KiCad schematic)
At the start: 1 part

Commit message: make board
Connections:
- net +3V3 renamed VIN
Changed lines of the file:
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@@
     (stroke (width 0) (type default))
+  )
+  (hierarchical_label "VIN" (shape input) (at 91.44 80.01 90) (fields_autoplaced)
+    (effects (font (size 1.27 1.27)) (justify left))
   )
   (hierarchical_label "SCL{slash}RX" (shape bidirectional) (at 76.2 88.9 180) (fields_autoplaced)
@@
         )
       )
-    )
-  )
-  (symbol (lib_id "power:+3V3") (at 91.44 80.01 0) (unit 1)
-    (in_bom yes) (on_board yes) (dnp no) (fields_autoplaced)
-    (property "Reference" "#PWR011" (at 91.44 83.82 0)
-      (effects (font (size 1.27 1.27)) hide)
-    )
-    (property "Value" "+3V3" (at 91.44 74.93 0)
-      (effects (font (size 1.27 1.27)))
-    )
-    (property "Footprint" "" (at 91.44 80.01 0)
-      (effects (font (size 1.27 1.27)) hide)
-    )
-    (property "Datasheet" "" (at 91.44 80.01 0)
-      (effects (font (size 1.27 1.27)) hide)
-    )
-    (pin "1")
-    (instances
-      (project "balloon"
-        (path "/390c33b5-3f3b-4c86-a202-e8d785058178/7a54972a-968a-463e-adb5-1c7fa9e20455"
-          (reference "#PWR011") (unit 1)
-        )
-      )
