File: gps.kicad_sch (KiCad schematic)
At the start: 1 part

Commit message: make board
Parts:
- removed U5: ~, symbol balloon_lib:Qwiic-SAM-M8Q
Changed lines of the file:
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@@
 (kicad_sch (version 20230121) (generator eeschema)
   (paper "A4")
-  (junction (at 137.16 109.22) (diameter 0) (color 0 0 0 0)
-  )
-  (junction (at 139.7 109.22) (diameter 0) (color 0 0 0 0)
-  )
-  (junction (at 139.7 83.82) (diameter 0) (color 0 0 0 0)
-  )
-  (wire (pts (xy 128.27 91.44) (xy 130.81 91.44))
-    (stroke (width 0) (type default))
-  )
-  (wire (pts (xy 137.16 109.22) (xy 139.7 109.22))
-    (stroke (width 0) (type default))
-  )
-  (wire (pts (xy 154.94 91.44) (xy 151.13 91.44))
-    (stroke (width 0) (type default))
-  )
-  (wire (pts (xy 139.7 109.22) (xy 142.24 109.22))
-    (stroke (width 0) (type default))
-  )
-  (wire (pts (xy 128.27 93.98) (xy 130.81 93.98))
-    (stroke (width 0) (type default))
-  )
-  (wire (pts (xy 128.27 100.33) (xy 130.81 100.33))
-    (stroke (width 0) (type default))
-  )
-  (wire (pts (xy 154.94 97.79) (xy 151.13 97.79))
-    (stroke (width 0) (type default))
-  )
-  (wire (pts (xy 139.7 83.82) (xy 142.24 83.82))
-    (stroke (width 0) (type default))
-  )
-  (wire (pts (xy 154.94 95.25) (xy 151.13 95.25))
-    (stroke (width 0) (type default))
-  )
-  (wire (pts (xy 154.94 100.33) (xy 151.13 100.33))
-    (stroke (width 0) (type default))
-  )
-  (wire (pts (xy 128.27 97.79) (xy 130.81 97.79))
-    (stroke (width 0) (type default))
-  )
-  (hierarchical_label "PPS" (shape output) (at 154.94 91.44 0) (fields_autoplaced)
-    (effects (font (size 1.27 1.27)) (justify left))
-  )
-  (hierarchical_label "RST_N" (shape input) (at 154.94 95.25 0) (fields_autoplaced)
-    (effects (font (size 1.27 1.27)) (justify left))
-  )
-  (hierarchical_label "INT" (shape output) (at 154.94 100.33 0) (fields_autoplaced)
-    (effects (font (size 1.27 1.27)) (justify left))
-  )
-  (hierarchical_label "RX" (shape input) (at 128.27 93.98 180) (fields_autoplaced)
-    (effects (font (size 1.27 1.27)) (justify right))
-  )
-  (hierarchical_label "SAFE_N" (shape input) (at 154.94 97.79 0) (fields_autoplaced)
-    (effects (font (size 1.27 1.27)) (justify left))
-  )
-  (hierarchical_label "SCL" (shape bidirectional) (at 128.27 100.33 180) (fields_autoplaced)
-    (effects (font (size 1.27 1.27)) (justify right))
-  )
-  (hierarchical_label "SDA" (shape bidirectional) (at 128.27 97.79 180) (fields_autoplaced)
-    (effects (font (size 1.27 1.27)) (justify right))
-  )
-  (hierarchical_label "TX" (shape output) (at 128.27 91.44 180) (fields_autoplaced)
-    (effects (font (size 1.27 1.27)) (justify right))
-  )
-  (symbol (lib_id "balloon_lib:Qwiic-SAM-M8Q") (at 139.7 96.52 0) (unit 1)
-    (in_bom yes) (on_board yes) (dnp no)
-    (property "Reference" "U5" (at 147.32 109.22 0)
-      (effects (font (size 1.27 1.27)) (justify left))
-    )
-    (property "Value" "~" (at 134.62 99.06 0)
-      (effects (font (size 1.27 1.27)))
-    )
-    (property "Footprint" "" (at 134.62 99.06 0)
-      (effects (font (size 1.27 1.27)) hide)
-    )
-    (property "Datasheet" "" (at 134.62 99.06 0)
-      (effects (font (size 1.27 1.27)) hide)
-    )
-    (pin "1")
-    (pin "10")
-    (pin "11")
-    (pin "12")
-    (pin "13")
-    (pin "14")
-    (pin "2")
-    (pin "3")
-    (pin "4")
-    (pin "5")
-    (pin "6")
-    (pin "7")
-    (pin "8")
-    (pin "9")
-    (instances
-      (project "balloon"
-        (path "/390c33b5-3f3b-4c86-a202-e8d785058178/c0965308-4fb8-43da-992f-faea07bd98c3"
-          (reference "U5") (unit 1)
-        )
-      )
-    )
-  )
-  (symbol (lib_id "power:+3V3") (at 139.7 83.82 0) (unit 1)
-    (in_bom yes) (on_board yes) (dnp no) (fields_autoplaced)
-    (property "Reference" "#PWR018" (at 139.7 87.63 0)
-      (effects (font (size 1.27 1.27)) hide)
-    )
-    (property "Value" "+3V3" (at 139.7 78.74 0)
-      (effects (font (size 1.27 1.27)))
-    )
-    (property "Footprint" "" (at 139.7 83.82 0)
-      (effects (font (size 1.27 1.27)) hide)
-    )
-    (property "Datasheet" "" (at 139.7 83.82 0)
-      (effects (font (size 1.27 1.27)) hide)
-    )
-    (pin "1")
-    (instances
-      (project "balloon"
-        (path "/390c33b5-3f3b-4c86-a202-e8d785058178/c0965308-4fb8-43da-992f-faea07bd98c3"
-          (reference "#PWR018") (unit 1)
-        )
-      )
-    )
-  )
-  (symbol (lib_id "power:GND1") (at 137.16 109.22 0) (unit 1)
-    (in_bom yes) (on_board yes) (dnp no) (fields_autoplaced)
-    (property "Reference" "#PWR017" (at 137.16 115.57 0)
-      (effects (font (size 1.27 1.27)) hide)
-    )
-    (property "Value" "GND1" (at 137.16 114.3 0)
-      (effects (font (size 1.27 1.27)))
-    )
-    (property "Footprint" "" (at 137.16 109.22 0)
-      (effects (font (size 1.27 1.27)) hide)
-    )
-    (property "Datasheet" "" (at 137.16 109.22 0)
-      (effects (font (size 1.27 1.27)) hide)
-    )
-    (pin "1")
-    (instances
-      (project "balloon"
-        (path "/390c33b5-3f3b-4c86-a202-e8d785058178/c0965308-4fb8-43da-992f-faea07bd98c3"
-          (reference "#PWR017") (unit 1)
-        )
-      )
-    )
-  )
 )
