File: balloon.kicad_sch (KiCad schematic)
At the start: 43 parts, among them J1 USB_B_Micro, J2 Conn_01x06_Socket, J3 Conn_01x06_Socket, J4 Conn_01x02_Socket, J5 Writing Connector, J7 Conn_01x06_Socket, SW1 DTS-63-F-N-V-RED, U1 CH340N, U3 AE_BME280, U4 AE_BNO055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

Commit message: add communication
Parts:
- removed C1: 100n, Capacitor_SMD:C_0603_1608Metric_Pad1.08x0.95mm_HandSolder, symbol Device:C
- removed J1: USB_B_Micro, Connector_USB:USB_Micro-B_Molex_47346-0001, symbol Connector:USB_B_Micro
- removed U1: CH340N, Package_SO:SOP-8_3.9x4.9mm_P1.27mm, symbol balloon_lib:CH340N
- added J1: Conn_01x03_Pin, symbol Connector:Conn_01x03_Pin
- added J12: Jack-DC, symbol Connector:Jack-DC
Connections:
- net GND1: now also J1.3 (Pin_3), J12.2
- net USART2_RX: now also J1.1 (Pin_1)
- net USART2_TX: now also J1.2 (Pin_2)
- new net PowerSource/12VDC: J12.1
- no-connect marks 8 -> 5
Other:
- sheet PowerSource ports: added 12VDC; removed 5VIN
