File: maxm10-s.kicad_sch (KiCad schematic)
At the start: 8 parts, among them J9 Conn_Coaxial, U11 MAX-M10S

Commit message: change conn
Parts:
- added J10: Conn_01x03_Socket, Connector_PinHeader_2.54mm:PinHeader_1x03_P2.54mm_Vertical, symbol Connector:Conn_01x03_Socket
- J9: footprint Connector_Coaxial:SMA_Amphenol_132291_Vertical -> Connector_Coaxial:U.FL_Hirose_U.FL-R-SMT-1_Vertical
- L1: footprint Resistor_SMD:R_0603_1608Metric_Pad0.98x0.95mm_HandSolder -> Resistor_SMD:R_0402_1005Metric_Pad0.72x0.64mm_HandSolder
Connections:
- net GND1: now also J10.3 (Pin_3)
- net RXD: now also J10.1 (Pin_1)
- net TXD: now also J10.2 (Pin_2)
Changed lines of the file:
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@@
   (junction (at 168.91 97.79) (diameter 0) (color 0 0 0 0)
   )
+  (junction (at 123.19 90.17) (diameter 0) (color 0 0 0 0)
+  )
   (junction (at 166.37 97.79) (diameter 0) (color 0 0 0 0)
+  )
+  (junction (at 125.73 87.63) (diameter 0) (color 0 0 0 0)
   )
   (junction (at 166.37 78.74) (diameter 0) (color 0 0 0 0)
@@
   (no_connect (at 128.27 97.79))
   (no_connect (at 128.27 110.49))
+  (wire (pts (xy 123.19 90.17) (xy 123.19 69.85))
+    (stroke (width 0) (type default))
+  )
   (wire (pts (xy 166.37 97.79) (xy 168.91 97.79))
     (stroke (width 0) (type default))
@@
     (stroke (width 0) (type default))
   )
-  (wire (pts (xy 119.38 87.63) (xy 128.27 87.63))
+  (wire (pts (xy 119.38 87.63) (xy 125.73 87.63))
     (stroke (width 0) (type default))
   )
@@
     (stroke (width 0) (type default))
   )
+  (wire (pts (xy 123.19 90.17) (xy 128.27 90.17))
+    (stroke (width 0) (type default))
+  )
   (wire (pts (xy 138.43 76.2) (xy 138.43 80.01))
     (stroke (width 0) (type default))
@@
     (stroke (width 0) (type default))
   )
+  (wire (pts (xy 116.84 72.39) (xy 114.3 72.39))
+    (stroke (width 0) (type default))
+  )
   (wire (pts (xy 148.59 80.01) (xy 148.59 78.74))
     (stroke (width 0) (type default))
@@
     (stroke (width 0) (type default))
   )
+  (wire (pts (xy 125.73 87.63) (xy 128.27 87.63))
+    (stroke (width 0) (type default))
+  )
   (wire (pts (xy 168.91 97.79) (xy 177.8 97.79))
     (stroke (width 0) (type default))
   )
+  (wire (pts (xy 125.73 67.31) (xy 125.73 87.63))
+    (stroke (width 0) (type default))
+  )
   (wire (pts (xy 138.43 80.01) (xy 140.97 80.01))
     (stroke (width 0) (type default))
   )
+  (wire (pts (xy 114.3 67.31) (xy 125.73 67.31))
+    (stroke (width 0) (type default))
+  )
+  (wire (pts (xy 123.19 69.85) (xy 114.3 69.85))
+    (stroke (width 0) (type default))
+  )
   (wire (pts (xy 143.51 116.84) (xy 143.51 115.57))
     (stroke (width 0) (type default))
@@
     (stroke (width 0) (type default))
   )
-  (wire (pts (xy 119.38 90.17) (xy 128.27 90.17))
+  (wire (pts (xy 119.38 90.17) (xy 123.19 90.17))
     (stroke (width 0) (type default))
   )
@@
         (path "/390c33b5-3f3b-4c86-a202-e8d785058178/ead08d60-297a-4e47-87a3-d098dce845f3"
           (reference "C21") (unit 1)
+        )
+      )
+    )
+  )
+  (symbol (lib_id "Connector:Conn_01x03_Socket") (at 109.22 69.85 0) (mirror y) (unit 1)
+    (in_bom yes) (on_board yes) (dnp no)
+    (property "Reference" "J10" (at 108.5088 68.6379 0)
+      (effects (font (size 1.27 1.27)) (justify left))
+    )
+    (property "Value" "Conn_01x03_Socket" (at 108.5088 71.0621 0)
+      (effects (font (size 1.27 1.27)) (justify left))
+    )
+    (property "Footprint" "Connector_PinHeader_2.54mm:PinHeader_1x03_P2.54mm_Vertical" (at 109.22 69.85 0)
+      (effects (font (size 1.27 1.27)) hide)
+    )
+    (property "Datasheet" "~" (at 109.22 69.85 0)
+      (effects (font (size 1.27 1.27)) hide)
+    )
+    (pin "1")
+    (pin "2")
+    (pin "3")
+    (instances
+      (project "balloon"
+        (path "/390c33b5-3f3b-4c86-a202-e8d785058178/ead08d60-297a-4e47-87a3-d098dce845f3"
+          (reference "J10") (unit 1)
         )
       )
@@
       (effects (font (size 1.27 1.27)))
     )
-    (property "Footprint" "Connector_Coaxial:SMA_Amphenol_132291_Vertical" (at 182.88 97.79 0)
+    (property "Footprint" "Connector_Coaxial:U.FL_Hirose_U.FL-R-SMT-1_Vertical" (at 182.88 97.79 0)
       (effects (font (size 1.27 1.27)) hide)
     )
@@
       (effects (font (size 1.27 1.27)) (justify left))
     )
-    (property "Footprint" "Resistor_SMD:R_0603_1608Metric_Pad0.98x0.95mm_HandSolder" (at 166.37 85.09 0)
+    (property "Footprint" "Resistor_SMD:R_0402_1005Metric_Pad0.72x0.64mm_HandSolder" (at 166.37 85.09 0)
       (effects (font (size 1.27 1.27)) hide)
     )
@@
         )
       )
+    )
+  )
+  (symbol (lib_id "power:GND1") (at 116.84 72.39 0) (unit 1)
+    (in_bom yes) (on_board yes) (dnp no) (fields_autoplaced)
+    (property "Reference" "#PWR01" (at 116.84 78.74 0)
+      (effects (font (size 1.27 1.27)) hide)
+    )
+    (property "Value" "GND1" (at 116.84 77.47 0)
+      (effects (font (size 1.27 1.27)))
+    )
+    (property "Footprint" "" (at 116.84 72.39 0)
+      (effects (font (size 1.27 1.27)) hide)
+    )
+    (property "Datasheet" "" (at 116.84 72.39 0)
+      (effects (font (size 1.27 1.27)) hide)
+    )
+    (pin "1")
+    (instances
+      (project "balloon"
+        (path "/390c33b5-3f3b-4c86-a202-e8d785058178"
+          (reference "#PWR01") (unit 1)
+        )
+        (path "/390c33b5-3f3b-4c86-a202-e8d785058178/a8964fff-36f8-4d65-a455-a6f79e0406e2"
+          (reference "#PWR020") (unit 1)
+        )
+        (path "/390c33b5-3f3b-4c86-a202-e8d785058178/ead08d60-297a-4e47-87a3-d098dce845f3"
+          (reference "#PWR059") (unit 1)
+        )
+      )

Commit message: change schematics
Parts:
- added J11: Conn_01x06_Socket, Connector_PinHeader_2.54mm:PinHeader_1x06_P2.54mm_Vertical, symbol Connector:Conn_01x06_Socket
Connections:
- net GND1: now also J11.1 (Pin_1), J11.2 (Pin_2)
- net RXD: now also J11.4 (Pin_4)
- net TXD: now also J11.5 (Pin_5)
- net VIN: now also J11.3 (Pin_3)
- no-connect marks 5 -> 6
Changed lines of the file:
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@@
   (junction (at 166.37 97.79) (diameter 0) (color 0 0 0 0)
   )
+  (junction (at 166.37 147.32) (diameter 0) (color 0 0 0 0)
+  )
   (junction (at 125.73 87.63) (diameter 0) (color 0 0 0 0)
   )
@@
   )
   (no_connect (at 128.27 95.25))
+  (no_connect (at 166.37 157.48))
   (no_connect (at 158.75 92.71))
   (no_connect (at 201.93 78.74))
@@
     (stroke (width 0) (type default))
   )
+  (wire (pts (xy 165.1 154.94) (xy 166.37 154.94))
+    (stroke (width 0) (type default))
+  )
   (wire (pts (xy 182.88 104.14) (xy 182.88 102.87))
     (stroke (width 0) (type default))
@@
     (stroke (width 0) (type default))
   )
+  (wire (pts (xy 156.21 147.32) (xy 166.37 147.32))
+    (stroke (width 0) (type default))
+  )
   (wire (pts (xy 148.59 80.01) (xy 148.59 78.74))
     (stroke (width 0) (type default))
@@
     (stroke (width 0) (type default))
   )
+  (wire (pts (xy 166.37 147.32) (xy 166.37 144.78))
+    (stroke (width 0) (type default))
+  )
+  (wire (pts (xy 165.1 149.86) (xy 166.37 149.86))
+    (stroke (width 0) (type default))
+  )
   (wire (pts (xy 143.51 76.2) (xy 143.51 80.01))
     (stroke (width 0) (type default))
   )
   (wire (pts (xy 168.91 106.68) (xy 168.91 116.84))
+    (stroke (width 0) (type default))
+  )
+  (wire (pts (xy 165.1 152.4) (xy 166.37 152.4))
     (stroke (width 0) (type default))
   )
@@
     (effects (font (size 1.27 1.27)) (justify right))
   )
+  (hierarchical_label "TXD" (shape output) (at 165.1 154.94 180) (fields_autoplaced)
+    (effects (font (size 1.27 1.27)) (justify right))
+  )
   (hierarchical_label "VIN" (shape input) (at 138.43 76.2 90) (fields_autoplaced)
     (effects (font (size 1.27 1.27)) (justify left))
@@
   )
   (hierarchical_label "RESET" (shape input) (at 125.73 107.95 180) (fields_autoplaced)
+    (effects (font (size 1.27 1.27)) (justify right))
+  )
+  (hierarchical_label "VIN" (shape input) (at 165.1 149.86 180) (fields_autoplaced)
+    (effects (font (size 1.27 1.27)) (justify right))
+  )
+  (hierarchical_label "RXD" (shape input) (at 165.1 152.4 180) (fields_autoplaced)
     (effects (font (size 1.27 1.27)) (justify right))
   )
@@
         (path "/390c33b5-3f3b-4c86-a202-e8d785058178/ead08d60-297a-4e47-87a3-d098dce845f3"
           (reference "#PWR058") (unit 1)
+        )
+      )
+    )
+  )
+  (symbol (lib_id "Connector:Conn_01x06_Socket") (at 171.45 149.86 0) (unit 1)
+    (in_bom yes) (on_board yes) (dnp no) (fields_autoplaced)
+    (property "Reference" "J11" (at 172.72 149.86 0)
+      (effects (font (size 1.27 1.27)) (justify left))
+    )
+    (property "Value" "Conn_01x06_Socket" (at 172.72 152.4 0)
+      (effects (font (size 1.27 1.27)) (justify left))
+    )
+    (property "Footprint" "Connector_PinHeader_2.54mm:PinHeader_1x06_P2.54mm_Vertical" (at 171.45 149.86 0)
+      (effects (font (size 1.27 1.27)) hide)
+    )
+    (property "Datasheet" "~" (at 171.45 149.86 0)
+      (effects (font (size 1.27 1.27)) hide)
+    )
+    (pin "1")
+    (pin "2")
+    (pin "3")
+    (pin "4")
+    (pin "5")
+    (pin "6")
+    (instances
+      (project "balloon"
+        (path "/390c33b5-3f3b-4c86-a202-e8d785058178/ead08d60-297a-4e47-87a3-d098dce845f3"
+          (reference "J11") (unit 1)
         )
       )
@@
         )
       )
+    )
+  )
+  (symbol (lib_id "power:GND1") (at 156.21 147.32 0) (unit 1)
+    (in_bom yes) (on_board yes) (dnp no) (fields_autoplaced)
+    (property "Reference" "#PWR01" (at 156.21 153.67 0)
+      (effects (font (size 1.27 1.27)) hide)
+    )
+    (property "Value" "GND1" (at 156.21 152.4 0)
+      (effects (font (size 1.27 1.27)))
+    )
+    (property "Footprint" "" (at 156.21 147.32 0)
+      (effects (font (size 1.27 1.27)) hide)
+    )
+    (property "Datasheet" "" (at 156.21 147.32 0)
+      (effects (font (size 1.27 1.27)) hide)
+    )
+    (pin "1")
+    (instances
+      (project "balloon"
+        (path "/390c33b5-3f3b-4c86-a202-e8d785058178"
+          (reference "#PWR01") (unit 1)
+        )
+        (path "/390c33b5-3f3b-4c86-a202-e8d785058178/a8964fff-36f8-4d65-a455-a6f79e0406e2"
+          (reference "#PWR020") (unit 1)
+        )
+        (path "/390c33b5-3f3b-4c86-a202-e8d785058178/ead08d60-297a-4e47-87a3-d098dce845f3"
+          (reference "#PWR062") (unit 1)
+        )
+      )
