File: rm92a.kicad_sch (KiCad schematic)
At the start: 17 parts

Commit message: make board
Parts:
- R1, R2, R3, R4, R5, R6, R7, R8, R9: footprint (none) -> Resistor_SMD:R_0603_1608Metric_Pad0.98x0.95mm_HandSolder
- U2: value ~ -> RM92A; footprint (none) -> balloon:RM92A
Connections:
- net +3V3 renamed VIN

Commit message: add communication
Parts:
- renumbered R8 to R10, R7 to R11, R9 to R12, R8 to R13, R7 to R14, R7 to R15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
