File: sdcard.kicad_sch (KiCad schematic)
At the start: 7 parts, among them J1 Micro_SD_Card_Det_Hirose_DM3AT

Commit message: make board
Parts:
- removed J1: Micro_SD_Card_Det_Hirose_DM3AT, symbol Connector:Micro_SD_Card_Det_Hirose_DM3AT
- added FB1, FB2, FB3, FB4, FB5, FB6: BLM18R, Resistor_SMD:R_0603_1608Metric_Pad0.98x0.95mm_HandSolder, symbol Device:FerriteBead_Small
- added J6: Micro_SD_Card_Det_Hirose_DM3AT, Connector_Card:microSD_HC_Hirose_DM3AT-SF-PEJM5, symbol Connector:Micro_SD_Card_Det_Hirose_DM3AT
- R22: renamed from R17; footprint (none) -> Resistor_SMD:R_0603_1608Metric_Pad0.98x0.95mm_HandSolder
- R23: renamed from R18; footprint (none) -> Resistor_SMD:R_0603_1608Metric_Pad0.98x0.95mm_HandSolder
- R24: renamed from R19; footprint (none) -> Resistor_SMD:R_0603_1608Metric_Pad0.98x0.95mm_HandSolder
- R25: renamed from R20; footprint (none) -> Resistor_SMD:R_0603_1608Metric_Pad0.98x0.95mm_HandSolder
- R26: renamed from R21; footprint (none) -> Resistor_SMD:R_0603_1608Metric_Pad0.98x0.95mm_HandSolder
- R27: renamed from R22; footprint (none) -> Resistor_SMD:R_0603_1608Metric_Pad0.98x0.95mm_HandSolder
Connections:
- net CLK: now also FB4.1
- net CMD: now also FB3.1
- net DAT0: now also FB5.1
- net DAT1: now also FB6.1
- net DAT2: now also FB1.1
- net DAT3: now also FB2.1
- net DET: now also J6.9 (DET_B)
- net GND1: now also J6.11 (SHIELD), J6.6 (VSS)
- net at R22.2: now also J6.10 (DET_A)
- net +3V3 renamed VIN
- net VIN: now also J6.4 (VDD)
- new net: FB4.2, J6.5 (CLK)
- new net: FB1.2, J6.1 (DAT2)
- new net: FB3.2, J6.3 (CMD)
- new net: FB2.2, J6.2 (DAT3/CD)
- new net: FB5.2, J6.7 (DAT0)
- new net: FB6.2, J6.8 (DAT1)
